File: NEO_R2_Schematic.brd (EAGLE design)
At the start: 55 x 100 mm, 30 parts, among them IC1 7805TV, IC2 4010N, J1 CON_TERMINAL_BLOCK_02-5MM, J2 CON_TERMINAL_BLOCK_02-5MM, J3 CON_TERMINAL_BLOCK_02-5MM, J4 CON_TERMINAL_BLOCK_02-5MM, U1 W25Q32FV

Commit message: BOM
Connections:
- net 3V: no longer IC2.16
- net 5V: now also IC2.16
Changed lines of the file:
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@@
 <setting verticaltext="up"/>
 </settings>
-<grid distance="1" unitdist="mm" unit="mm" style="lines" multiple="1" display="yes" altdistance="1" altunitdist="mil" altunit="mm"/>
+<grid distance="10" unitdist="mm" unit="mm" style="lines" multiple="1" display="yes" altdistance="1" altunitdist="mil" altunit="mm"/>
 <layers>
 <layer number="1" name="Top" color="4" fill="1" visible="yes" active="yes"/>
@@
 </signal>
 <signal name="3V">
-<contactref element="IC2" pad="16"/>
 <contactref element="ARDUINO_NANO1" pad="2"/>
 <contactref element="U1" pad="8"/>
@@
 <wire x1="24.5142" y1="51.4858" x2="25.0698" y2="51.4858" width="0.5" layer="1"/>
 <wire x1="10.453" y1="65.547" x2="24.5142" y2="51.4858" width="0.5" layer="1"/>
-<wire x1="25.0698" y1="51.4858" x2="28.3972" y2="48.1584" width="0.5" layer="1"/>
-<wire x1="28.3972" y1="48.1584" x2="28.3972" y2="47.2948" width="0.5" layer="1"/>
 <wire x1="25.0698" y1="51.4858" x2="20.8788" y2="47.2948" width="0.5" layer="1"/>
 <wire x1="20.8788" y1="47.2948" x2="20.7772" y2="47.2948" width="0.5" layer="1"/>
-<wire x1="28.3972" y1="47.2948" x2="31.4452" y2="47.2948" width="0.5" layer="1"/>
 <wire x1="31.4452" y1="47.2948" x2="31.75" y2="46.99" width="0.5" layer="1"/>
 <wire x1="35.48823125" y1="46.6852" x2="37.0078" y2="46.6852" width="0.5" layer="1"/>
@@
 <wire x1="46" y1="94.5" x2="51.77" y2="94.5" width="0.5" layer="16"/>
 <wire x1="39" y1="101.5" x2="46" y2="94.5" width="0.5" layer="16"/>
+<wire x1="31.75" y1="46.99" x2="30.2964" y2="48.4436" width="0.508" layer="1"/>
+<wire x1="30.2964" y1="48.4436" x2="28.76953125" y2="48.4436" width="0.508" layer="1"/>
+<wire x1="25.72733125" y1="51.4858" x2="25.0698" y2="51.4858" width="0.508" layer="1"/>
+<wire x1="28.76953125" y1="48.4436" x2="25.72733125" y2="51.4858" width="0.508" layer="1"/>
 </signal>
 <signal name="12V">
@@
 </polygon>
 <contactref element="X4" pad="1"/>
+<contactref element="IC2" pad="16"/>
 </signal>
 <signal name="N$2">
