File: NEO_R2_Schematic.sch (EAGLE design)
At the start: 30 parts, among them IC1 7805TV, IC2 4010N, J1 CON_TERMINAL_BLOCK_02-5MM, J2 CON_TERMINAL_BLOCK_02-5MM, J3 CON_TERMINAL_BLOCK_02-5MM, J4 CON_TERMINAL_BLOCK_02-5MM, U1 W25Q32FV

Commit message: BOM
Connections:
- net 5V: now also IC2P.VDD
Changed lines of the file:
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@@
 <pinref part="SUPPLY5" gate="G$1" pin="5V"/>
+</segment>
+<segment>
+<pinref part="IC2" gate="P" pin="VDD"/>
+<wire x1="363.22" y1="172.72" x2="363.22" y2="180.34" width="0.1524" layer="91"/>
+<label x="363.22" y="175.26" size="1.778" layer="95" rot="R90"/>
 </segment>
 </net>
